File: PTP_LV.kicad_sch (KiCad schematic)
At the start: 0 parts

Commit message: dodan naziv i ostali opisi projekta
Other:
- company: (none) -> TVZ - Tehničko veleučilište u Zagrebu
- title: (none) -> BCD brojač
Changed lines of the file:
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@@
 	(generator_version "9.0")
 	(paper "A4")
+	(title_block
+		(title "BCD brojač")
+		(date "2025-10-20")
+		(rev "0")
+		(company "TVZ - Tehničko veleučilište u Zagrebu")
+		(comment 1 "Izradio: Dean Fraj")
+	)
 	(sheet_instances
 		(path "/"
